File: bluescsi/kicad/HDB50_External/HDB50_External.kicad_sch (KiCad schematic)
At the start: 57 parts, among them J2 5749084-5, U3 AMS1117-2.85, U4 LVT245, U5 LVT125, U6 LVT125, U7 LVT125, U9 LVT245

Commit message: Add HD50_External.svg
Other:
- note removed: "BlueSCSI © Eric Helgeson PCB © Tech by Androda, LLC Licensed under CERN-OHL-S v2 https://ohwr.org/cern_ohl_s_v2.txt"
- note removed: "This source is distributed WITHOUT ANY EXPRESS OR IMPLIED WARRANTY, INCLUDING OF MERCHANTABILITY, SATISFACTORY QUALITY AND FITNESS FOR A PARTICULAR PURPOSE. Please see the CERN-OHL-S v2 for applicable conditions. As per CERN-OHL-S v2 section 4, should You produce hardware based on this source, You must where practicable maintain the Source Location visible on the external case of the Device or ot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"
Changed lines of the file:
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@@
-		)
-	)
-	(text "BlueSCSI © Eric Helgeson\nPCB © Tech by Androda, LLC\n\nLicensed under CERN-OHL-S v2\nhttps://ohwr.org/cern_ohl_s_v2.txt"
-		(exclude_from_sim no)
-		(at 229.108 174.244 0)
-		(effects
-			(font
-				(size 1.27 1.27)
-			)
 		)
 	)
@@
 		)
 	)
-	(text "This source is distributed WITHOUT ANY EXPRESS OR IMPLIED WARRANTY,          \nINCLUDING OF MERCHANTABILITY, SATISFACTORY QUALITY AND FITNESS FOR A         \nPARTICULAR PURPOSE. Please see the CERN-OHL-S v2 for applicable conditions.\n\nAs per CERN-OHL-S v2 section 4, should You produce hardware based on this    \nsource, You must where practicable maintain the Source Location visible      \non the external case of the Device or other products you make using this source.  \n"
-		(exclude_from_sim no)
-		(at 233.68 210.058 0)
-		(effects
-			(font
-				(size 1.27 1.27)
-			)
-		)
-	)
